File: pcb/mekko5X/mekko5X.kicad_pcb (KiCad board)
At the start: 2 copper layers, 190.5 x 131 mm, 98 parts, among them SW1 RotaryEncoder_Switch, SW10 SW_SPST, SW11 SW_SPST, SW12 SW_SPST, SW13 SW_SPST, SW14 SW_SPST, SW15 SW_SPST, SW16 SW_SPST, SW17 SW_SPST, SW18 SW_SPST, SW19 SW_SPST, SW2 RotaryEncoder_Switch, SW20 SW_SPST, SW21 SW_SPST, SW22 SW_SPST, SW23 SW_SPST, SW24 SW_SPST, SW25 SW_SPST, SW26 SW_SPST, SW27 SW_SPST, SW28 SW_SPST, SW29 SW_SPST, SW3 SW_SPST, SW30 SW_SPST, SW31 SW_SPST, SW32 SW_SPST, SW33 SW_SPST, SW34 SW_SPST, SW35 SW_SPST, SW36 SW_SPST, SW37 SW_SPST, SW38 SW_SPST, SW39 SW_SPST, SW4 SW_SPST, SW40 SW_SPST, SW41 SW_SPST, SW42 SW_SPST, SW44 SW_SPST, SW5 SW_SPST, SW6 SW_SPST, SW7 SW_SPST, SW8 SW_SPST, SW9 SW_SPST, U1 SSD1309, U2 SSD1309, U3 Pico

Commit message: add files
Routing:
- net cs1: track 23.4 -> 40.9 mm, vias 0 -> 2
- net cs2: track 102.4 -> 118.8 mm, vias 0 -> 2
- net dc: track 116.3 -> 106.6 mm
- net 3v3: track 142.3 -> 151.9 mm
- net sclk: track 113.3 -> 118.1 mm
- net res: track 111.5 -> 106.7 mm
- net gnd: track 166.6 -> 167.4 mm, vias 3 -> 4
Other:
- board text added: "mekko5x v0.1 by sporewoh"
- board text removed: "mekko5x v0.0 by sporewoh"
